File: pcb/kicad/quad.kicad_pcb (KiCad board)
At the start: 2 copper layers, 75.1 x 75.1 mm, 134 parts, among them CN1 CN1, CN2 CN2, CN3 CN3, CN4 CN4, CN5 CN5, Q1 AO3400A, Q2 AO3400A, Q3 AO3400A, Q4 AO3400A, SW1 SW1, SW2 SW2, U1 ESP32-S3-WROOM-1-N16R8, U2 BMI323, U3 TLV75733PDBVR, U4 TP4054-42-SOT25R

Commit message: Replace 3.3 V LDO with TPS63001 buck-boost against brown-outs, fix drill slots/silk/KiCad schematic, add firmware battery and arming safety
Parts:
- removed the ? at (95.1, 107.6)
- removed the ? at (92.7, 97.5)
- removed the ? at (88.7, 106.0)
- removed the ? at (89.7, 80.5)
- removed the ? at (93.6, 107.6)
- removed the ? at (94.7, 103.2)
- removed the ? at (93.7, 103.2)
- removed the ? at (88.9, 109.4)
- added ?: , tscircuit:Unknown, F.Cu at (90.4, 80.1)
- added ?: , tscircuit:Unknown, F.Cu at (94.0, 108.8)
- added ?: , tscircuit:Unknown, F.Cu at (93.8, 108.0)
- added ?: , tscircuit:Unknown, F.Cu at (94.0, 100.0)
- added ?: , tscircuit:Unknown, F.Cu at (93.8, 104.5)
- added ?: , tscircuit:Unknown, F.Cu at (94.0, 103.8)
- added ?: , tscircuit:Unknown, F.Cu at (96.0, 97.5)
- added C13: 22uF, tscircuit:capacitor_cap0603, F.Cu at (88.7, 80.2)
- added L1: 2.2µH, tscircuit:FTC252012S2R2MBCA, F.Cu at (89.5, 106.3)
- added R21: 100Ω, tscircuit:resistor_res0402, F.Cu at (95.2, 109.0)
- C2: value 22uF -> 100nF; footprint tscircuit:capacitor_cap0603 -> tscircuit:capacitor_cap0402
- C7: value 10uF -> 22uF
- U3: value TLV75733PDBVR -> TPS63001DRCR; footprint tscircuit:TLV75733PDBVR -> tscircuit:TPS63001DRCR
- moved C7 2.54 mm to (92.2, 103.8), turned to 0 degrees
- moved C6 2.51 mm to (92.2, 108.8), turned to 0 degrees
- moved U3 2.02 mm to (93.0, 106.3), turned to 0 degrees
- moved C2 1.15 mm to (95.9, 106.7), turned to 90 degrees
- moved C10 0.55 mm to (94.5, 101.3), turned to 90 degrees
- moved R20 0.54 mm to (93.5, 101.3), turned to 90 degrees
Connections:
- C2 pad 1: V3V3 -> VINA
- U3 pad 1: VBAT -> V3V3
- U3 pad 2: GND -> LX2
- U3 pad 3: VBAT -> GND
- U3 pad 4: (no net) -> LX1
- U3 pad 5: V3V3 -> VBAT
Routing:
- net GND: track 70.8 -> 83.7 mm, vias 42 -> 41
- net VBAT: track 164.6 -> 153.2 mm
- net V3V3: track 75.7 -> 82.0 mm
- net VINA: track 0.00 -> 5.77 mm
- net LX1: track 0.00 -> 2.10 mm
- net LX2: track 0.00 -> 2.10 mm
- net USB_DP: track 26.8 -> 28.2 mm
- net USB_DN: track 23.8 -> 24.8 mm
- net VSENSE: track 7.87 -> 7.07 mm

Commit message: Move motor connectors out to the May 2026 position (as far along the arms as their tabs allow)
Parts:
- moved CN1 1.56 mm to (117.6, 82.4)
- moved CN2 1.56 mm to (117.6, 117.6)
- moved CN3 1.56 mm to (82.4, 117.6)
- moved CN4 1.56 mm to (82.4, 82.4)
Routing:
- net VBAT: track 153.2 -> 159.4 mm
- net M3: track 6.84 -> 8.38 mm
- net M2: track 6.84 -> 8.38 mm
- net M1: track 6.84 -> 8.38 mm
- net M0: track 6.84 -> 8.38 mm

Commit message: Fix gaps from review: firmware safety (heartbeat, stuck/idle disarm, still-and-level calibration, no boot motor sweep, IMU config), BLE client hardening, BAT/polarity silkscreen, ordering and bring-up docs
Other:
- board text added: "BAT"
- board text added: "REV A 2026-09"
- board text removed: "+"
- board text removed: "-"
- board text removed: "rev A 2026-09"
Changed lines of the file:
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@@
+	)
+	(gr_line
+		(start 85.26 83.26)
+		(end 86.26 83.26)
+		(stroke
+			(width 0.2)
+			(type solid)
+		)
+		(layer "F.SilkS")
+	)
+	(gr_line
+		(start 85.26 116.74)
+		(end 86.26 116.74)
+		(stroke
+			(width 0.2)
+			(type solid)
+		)
+		(layer "F.SilkS")
+	)
+	(gr_line
+		(start 85.76 83.76)
+		(end 85.76 82.76)
+		(stroke
+			(width 0.2)
+			(type solid)
+		)
+		(layer "F.SilkS")
+	)
+	(gr_line
+		(start 85.76 117.24)
+		(end 85.76 116.24)
+		(stroke
+			(width 0.2)
+			(type solid)
+		)
+		(layer "F.SilkS")
 	)
 	(gr_line
@@
 		(stroke
 			(width 0.15)
+			(type solid)
+		)
+		(layer "F.SilkS")
+	)
+	(gr_line
+		(start 104.37 118.35)
+		(end 105.17 118.35)
+		(stroke
+			(width 0.2)
+			(type solid)
+		)
+		(layer "F.SilkS")
+	)
+	(gr_line
+		(start 104.77 118.75)
+		(end 104.77 117.95)
+		(stroke
+			(width 0.2)
+			(type solid)
+		)
+		(layer "F.SilkS")
+	)
+	(gr_line
+		(start 105.63 118.35)
+		(end 106.43 118.35)
+		(stroke
+			(width 0.2)
+			(type solid)
+		)
+		(layer "F.SilkS")
+	)
+	(gr_line
+		(start 113.74 83.26)
+		(end 114.74 83.26)
+		(stroke
+			(width 0.2)
+			(type solid)
+		)
+		(layer "F.SilkS")
+	)
+	(gr_line
+		(start 113.74 116.74)
+		(end 114.74 116.74)
+		(stroke
+			(width 0.2)
+			(type solid)
+		)
+		(layer "F.SilkS")
+	)
+	(gr_line
+		(start 114.24 83.76)
+		(end 114.24 82.76)
+		(stroke
+			(width 0.2)
+			(type solid)
+		)
+		(layer "F.SilkS")
+	)
+	(gr_line
+		(start 114.24 117.24)
+		(end 114.24 116.24)
+		(stroke
+			(width 0.2)
 			(type solid)
 		)
@@
 		)
 	)
-	(gr_text "RST"
-		(at 82.1 102.55 0)
+	(gr_text "M3 CW"
+		(at 71.5 71.5 -45)
 		(layer "F.SilkS")
 		(effects
 			(font
-				(size 1.05 1.05)
+				(size 1.225 1.225)
 				(thickness 0.16)
 			)
 		)
 	)
+	(gr_text "M1 CW"
+		(at 128.5 128.5 -45)
+		(layer "F.SilkS")
+		(effects
+			(font
+				(size 1.225 1.225)
+				(thickness 0.16)
+			)
+		)
+	)
+	(gr_text "RST"
+		(at 82.35 102.55 0)
+		(layer "F.SilkS")
+		(effects
+			(font
+				(size 1.225 1.225)
+				(thickness 0.16)
+			)
+		)
+	)
 	(gr_text "CHG"
 		(at 100.4 108.7 0)
@@
 		(effects
 			(font
-				(size 1.05 1.05)
+				(size 1.225 1.225)
 				(thickness 0.16)
 			)
 		)
 	)
-	(gr_text "+"
-		(at 85.76 83.26 0)
-		(layer "F.SilkS")
+	(gr_text "BAT"
+		(at 109.35 118.35 0)
+		(layer "F.SilkS")
+		(effects
+			(font
+				(size 1.225 1.225)
+				(thickness 0.16)
+			)
+		)
+	)
+	(gr_text "M2 CCW"
+		(at 71.5 128.5 45)
+		(layer "F.SilkS")
+		(effects
+			(font
+				(size 1.225 1.225)
+				(thickness 0.16)
+			)
+		)
+	)
+	(gr_text "M0 CCW"
+		(at 128.5 71.5 45)
+		(layer "F.SilkS")
+		(effects
+			(font
+				(size 1.225 1.225)
+				(thickness 0.16)
+			)
+		)
+	)
+	(gr_text "REV A 2026-09"
+		(at 100 95.7 0)
+		(layer "B.SilkS")
 		(effects
 			(font
@@
 				(thickness 0.16)
 			)
-		)
-	)
-	(gr_text "+"
-		(at 85.76 116.74 0)
-		(layer "F.SilkS")
-		(effects
-			(font
-				(size 1.12 1.12)
-				(thickness 0.16)
-			)
-		)
-	)
-	(gr_text "+"
-		(at 114.24 83.26 0)
-		(layer "F.SilkS")
-		(effects
-			(font
-				(size 1.12 1.12)
-				(thickness 0.16)
-			)
-		)
-	)
-	(gr_text "+"
-		(at 114.24 116.74 0)
-		(layer "F.SilkS")
-		(effects
-			(font
-				(size 1.12 1.12)
-				(thickness 0.16)
-			)
-		)
-	)
-	(gr_text "M3 CW"
-		(at 71.5 71.5 -45)
-		(layer "F.SilkS")
-		(effects
-			(font
-				(size 1.19 1.19)
-				(thickness 0.16)
-			)
-		)
-	)
-	(gr_text "M1 CW"
-		(at 128.5 128.5 -45)
-		(layer "F.SilkS")
-		(effects
-			(font
-				(size 1.19 1.19)
-				(thickness 0.16)
-			)
-		)
-	)
-	(gr_text "M2 CCW"
-		(at 71.5 128.5 45)
-		(layer "F.SilkS")
-		(effects
-			(font
-				(size 1.19 1.19)
-				(thickness 0.16)
-			)
-		)
-	)
-	(gr_text "M0 CCW"
-		(at 128.5 71.5 45)
-		(layer "F.SilkS")
-		(effects
-			(font
-				(size 1.19 1.19)
-				(thickness 0.16)
-			)
-		)
-	)
-	(gr_text "+"
-		(at 104.77 118.35 0)
-		(layer "F.SilkS")
-		(effects
-			(font
-				(size 1.26 1.26)
-				(thickness 0.162)
-			)
-		)
-	)
-	(gr_text "-"
-		(at 106.03 118.35 0)
-		(layer "F.SilkS")
-		(effects
-			(font
-				(size 1.26 1.26)
-				(thickness 0.162)
-			)
+			(justify mirror)
 		)
 	)
@@
 		(effects
 			(font
-				(size 1.05 1.05)
-				(thickness 0.16)
-			)
-			(justify mirror)
-		)
-	)
-	(gr_text "rev A  2026-09"
-		(at 100 96.6 0)
-		(layer "B.SilkS")
-		(effects
-			(font
-				(size 1.05 1.05)
+				(size 1.225 1.225)
 				(thickness 0.16)
 			)
@@
 		(effects
 			(font
-				(size 1.05 1.05)
+				(size 1.225 1.225)
 				(thickness 0.16)
 			)
@@
 		(effects
 			(font
-				(size 1.05 1.05)
+				(size 1.225 1.225)
 				(thickness 0.16)
 			)
@@
 		(effects
 			(font
-				(size 1.05 1.05)
+				(size 1.225 1.225)
 				(thickness 0.16)
 			)
@@
 		(effects
 			(font
-				(size 1.05 1.05)
+				(size 1.225 1.225)
 				(thickness 0.16)
 			)

Commit message: Rework flight control for a first real hover: flight.c (slow-corrected gravity estimate, angle-rate PID with lift-off-aware integrators) at 500 Hz on 800 Hz IMU data, arrow steering, trim and gain keys in NVS, hover simulator, client Esc fixes, R16 5.1k for 170/250 mAh packs
Parts:
- R16: value 3.3kΩ -> 5.1kΩ
Changed lines of the file:
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@@
 			)
 		)
-		(property "Value" "3.3kΩ"
+		(property "Value" "5.1kΩ"
 			(at 0 3 0)
 			(layer "F.Fab")
@@
 			)
 		)
-		(property "Supplier Part Number" "C25890"
+		(property "Supplier Part Number" "C25905"
 			(at 0 0 0)
 			(layer "F.Fab")
