File: pcb/kicad/quad.kicad_sch (KiCad schematic)
At the start: 57 parts, among them CN1 HC-1.25-2PWT, CN2 HC-1.25-2PWT, CN3 HC-1.25-2PWT, CN4 HC-1.25-2PWT, CN5 53398-0271, Q1 AO3400A, Q2 AO3400A, Q3 AO3400A, Q4 AO3400A, SW1 SW1, SW2 SW2, U1 ESP32-S3-WROOM-1-N16R8, U2 BMI323, U3 TLV75733PDBVR, U4 TP4054-42-SOT25R

Commit message: Replace 3.3 V LDO with TPS63001 buck-boost against brown-outs, fix drill slots/silk/KiCad schematic, add firmware battery and arming safety
Parts:
- removed U3: TLV75733PDBVR, symbol Device:U_TLV75733PDBVR
- added C13: 22uF, symbol Device:capacitor_down
- added L1: 2.2µH, symbol Device:inductor_right
- added R21: 100Ω, symbol Device:boxresistor_right
- added U3: TPS63001DRCR, symbol Device:U_TPS63001DRCR
- C2: value 22uF -> 100nF
- C7: value 10uF -> 22uF
Connections:
- net GND: now also C13.2, U3.11 (EP), U3.3 (PGND), U3.7 (PS), U3.9 (GND)
- net V3V3: now also C13.1, U3.1 (VOUT), U3.10 (FB); no longer C2.1
- net VBAT: now also R21.1, U3.5 (VIN)
- new net: L1.2, U3.2 (L2)
- new net: L1.1, U3.4 (L1)
- new net: C2.1, R21.2, U3.6 (EN), U3.8 (VINA)
- no-connect marks 42 -> 41
Other:
- note added: "3.3 V from 1.8-5.5 V in"
- note added: "EN on VINA: always on · PS/SYNC low: power-save mode"
- note added: "USB-C 5 V → TP4054 charges the 1S LiPo at 260 mA (R16 = 3.3 k, datasheet formula 1) · TPS63001 buck-boost makes 3.3 V from VBAT · ESP32-S3 drives four brushed motors through AO3400A low-side switches"
- note added: "bulk at the connector · C11, C12 at the motor rails · C6 at the converter"
- note removed: "EN tied to IN: on whenever a battery is in"
- note removed: "USB-C 5 V → TP4054 charges the 1S LiPo at 260 mA (R16 = 3.3 k, datasheet formula 1) · TLV757 makes 3.3 V from VBAT · ESP32-S3 drives four brushed motors through AO3400A low-side switches"
- note removed: "bulk at the connector · C11, C12 at the motor rails · C6 at the LDO"

Commit message: Rework flight control for a first real hover: flight.c (slow-corrected gravity estimate, angle-rate PID with lift-off-aware integrators) at 500 Hz on 800 Hz IMU data, arrow steering, trim and gain keys in NVS, hover simulator, client Esc fixes, R16 5.1k for 170/250 mAh packs
Parts:
- R16: value 3.3kΩ -> 5.1kΩ
Other:
- note added: "USB-C 5 V → TP4054 charges the 1S LiPo at 190 mA (R16 = 5.1 k, datasheet formula 1) · TPS63001 buck-boost makes 3.3 V from VBAT · ESP32-S3 drives four brushed motors through AO3400A low-side switches"
- note removed: "USB-C 5 V → TP4054 charges the 1S LiPo at 260 mA (R16 = 3.3 k, datasheet formula 1) · TPS63001 buck-boost makes 3.3 V from VBAT · ESP32-S3 drives four brushed motors through AO3400A low-side switches"
